Commit message: Modify my_robot to sawpn and removed from world file

File: Project2/catkin_ws/src/my_robot/urdf/my_robot.xacro (robot description, xacro)
@@ -9,5 +9,5 @@
   </joint>
   <link name='chassis'>
-    <pose>0 0 0.1 0 0 0</pose>
+   <pose>0 0 0.1 0 0 0</pose>
     <inertial>
       <mass value="15.0"/>
@@ -22,5 +22,5 @@
       <origin xyz="0 0 0" rpy="0 0 0"/>
       <geometry>
-        <box size=".4 .2 .1"/>
+        <cylinder radius="0.3" length="0.1"/>
       </geometry>
     </collision>
@@ -28,5 +28,5 @@
       <origin xyz="0 0 0" rpy="0 0 0"/>
       <geometry>
-        <box size=".4 .2 .1"/>
+        <cylinder radius="0.3" length="0.1"/>
       </geometry>
     </visual>
@@ -173,3 +173,12 @@
     <child link="hokuyo"/>
   </joint>
+  <gazebo reference="chassis">
+    <material>Gazebo/Orange</material>
+  </gazebo>
+  <gazebo reference="left_wheel">
+    <material>Gazebo/Turquoise</material>
+  </gazebo>
+  <gazebo reference="right_wheel">
+    <material>Gazebo/Turquoise</material>
+  </gazebo>
 </robot>
